Commit message: joint 6,7 추가 / urdf 중량 정보 추가
todo 중력보상 임피던스제어

File: right_arm_urdf/right_arm_urdf.urdf (robot description, URDF)
Before this commit: robot right_arm_urdf, 8 links, 7 joints
Links:
- link base_link: mass 9.776297041947103 -> 1.2
- link link_1: mass 2.9253509837230443 -> 1.1
- link link_2: mass 2.743489599560163 -> 1.1
- link link_3: mass 4.786828066244079 -> 0.9
- link link_4: mass 2.423118371436369 -> 0.7
- link link_5: mass 1.7450144413361988 -> 0.25
- link link_6: mass 5.753617330726645 -> 0.7
- link link_end: mass 2.4220783479433985 -> 0.5
