Commit message: 중력보상 수정 및 urdf 변경

File: right_urdf/right_urdf.urdf (robot description, URDF)
Before this commit: robot right_urdf, 8 links, 7 joints
Links:
- link base_link: mass 2.6289526754642267 -> 1.2
- link link_1: mass 2.9253509837230443 -> 1.1
- link link_2: mass 2.743489599560163 -> 1.0
- link link_3: mass 4.786828066244079 -> 1.1
- link link_4: mass 2.423118371436369 -> 0.6
- link link_5: mass 1.7450144413361988 -> 0.5
- link link_6: mass 0.2398006000337179 -> 0.8
- link link_end: mass 0.09931289188708475 -> 0.2
